File: jac_board.kicad_pcb (KiCad board)
At the start: 2 copper layers, 100 x 100 mm, 92 parts, among them J10 Conn_01x04_Female, J11 Conn_01x04_Female, J12 Conn_01x04_Female, J2 726386-2, J3 726386-2, J4 726386-2, J5 726386-2, J7 Screw_Terminal_01x04, J8 Screw_Terminal_01x04, J9 Screw_Terminal_01x02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

Commit message: Primer commit - Migracion de Kicad6 a Kicad7
Other:
- net class Default removed
