File: jac_board.kicad_sch (KiCad schematic)
At the start: 4 parts

Commit message: Planteamiento nuevo proeycto de mosquito - Se eelmiraon del esquematico las entradas a 0V y las salidas a Leds
Other:
- note added: "3.3v"
- note added: "4 Digital Input - 3.3-5V"
- note added: "4 ouputs 12V"
- note added: "ARDUINO"
- note added: "DEJAR RX/TX para conectar modulo RS232/485"
- note added: "RPI"
- note added: "awg18"
- note added: "distancia??"
Changed lines of the file:
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@@
 (kicad_sch (version 20230121) (generator eeschema)
   (paper "A4")
+  (wire (pts (xy 162.56 114.3) (xy 220.98 114.3))
+    (stroke (width 0) (type default))
+  )
+  (wire (pts (xy 162.56 123.19) (xy 220.98 123.19))
+    (stroke (width 0) (type default))
+  )
+  (wire (pts (xy 163.83 118.11) (xy 220.98 118.11))
+    (stroke (width 0) (type default))
+  )
+  (rectangle (start 93.98 106.68) (end 162.56 128.27)
+    (stroke (width 0) (type default))
+    (fill (type none))
+  )
+  (rectangle (start 220.98 106.68) (end 279.4 132.08)
+    (stroke (width 0) (type default))
+    (fill (type none))
+  )
+  (text "3.3v" (at 222.25 130.81 0)
+    (effects (font (size 6 6) (thickness 1.2) bold) (justify left bottom))
+  )
+  (text "4 ouputs 12V" (at 222.25 162.56 0)
+    (effects (font (size 6 6) (thickness 1.2) bold) (justify left bottom))
+  )
+  (text "RPI" (at 106.68 121.92 0)
+    (effects (font (size 6 6) (thickness 1.2) bold) (justify left bottom))
+  )
+  (text "3.3v" (at 143.51 127 0)
+    (effects (font (size 6 6) (thickness 1.2) bold) (justify left bottom))
+  )
+  (text "DEJAR RX/TX para conectar modulo RS232/485" (at 222.25 140.97 0)
+    (effects (font (size 6 6) (thickness 1.2) bold) (justify left bottom))
+  )
+  (text "4 Digital Input - 3.3-5V" (at 222.25 149.86 0)
+    (effects (font (size 6 6) (thickness 1.2) bold) (justify left bottom))
+  )
+  (text "distancia??" (at 166.37 113.03 0)
+    (effects (font (size 6 6) (thickness 1.2) bold) (justify left bottom))
+  )
+  (text "awg18" (at 175.26 102.87 0)
+    (effects (font (size 6 6) (thickness 1.2) bold) (justify left bottom))
+  )
+  (text "ARDUINO" (at 233.68 121.92 0)
+    (effects (font (size 6 6) (thickness 1.2) bold) (justify left bottom))
+  )
   (symbol (lib_id "Mechanical:MountingHole") (at 71.12 69.85 0) (unit 1)
     (in_bom yes) (on_board yes) (dnp no)
